Commit message: commit

File: mybot_description/urdf/rolstoelbot.xacro (robot description, xacro)
@@ -20,168 +20,23 @@
    <inertia ixx="0.1" iyy="0.1" izz="0.1" ixy="0" ixz="0" iyz="0" />
   </inertial>
-  <collision name='caster_collision_right'>
-      <origin xyz="-0.29 0.235 -0.54" rpy=" 0 0 0"/>
-      <geometry>
-        <sphere radius="0.1"/>
-      </geometry>
-      <surface>
-        <friction>
-          <ode>
-            <mu>0</mu>
-            <mu2>0</mu2>
-            <slip1>1.0</slip1>
-            <slip2>1.0</slip2>
-          </ode>
-        </friction>
-      </surface>
-    </collision>
-    <visual name='caster_collision_right_visual'>
-     <origin xyz="-0.29 0.235 -0.54" rpy=" 0 0 0"/>
-     <geometry>
-      <sphere radius="0.1"/>
-     </geometry>
-    </visual>
-    <collision name='caster_collision_left'>
-      <origin xyz="-0.29 -0.235 -0.54" rpy=" 0 0 0"/>
-      <geometry>
-        <sphere radius="0.1"/>
-      </geometry>
-      <surface>
-        <friction>
-          <ode>
-            <mu>0</mu>
-            <mu2>0</mu2>
-            <slip1>1.0</slip1>
-            <slip2>1.0</slip2>
-          </ode>
-        </friction>
-      </surface>
-    </collision>
-    <visual name='caster_collision_left_visual'>
-     <origin xyz="-0.29 -0.235 -0.54" rpy=" 0 0 0"/>
-     <geometry>
-      <sphere radius="0.1"/>
-     </geometry>
-    </visual>
- </link>
- <visual name='caster_front_visual'>
-  <origin xyz="-0.29 0.265 -0.56" rpy=" 0 0 0"/>
-  <geometry>
-    <sphere radius="0.1"/>
-  </geometry>
- </visual>
- <link name="front_wheel_left">
-  <visual>
-   <geometry>
-    <cylinder length="0.06" radius="0.16"/>
-   </geometry>
-   <material name="black"/>
-  </visual>
-  <collision>
-   <geometry>
-    <cylinder length="0.06" radius="0.16"/>
-   </geometry>
-  </collision>
-  <inertial>
-   <mass value="1.0" />
-   <inertia ixx="0.1" iyy="0.1" izz="0.1" ixy="0" ixz="0" iyz="0" />
-  </inertial>
- </link>
- <joint name="front_wheel_left_joint" type="continuous">
-  <axis xyz="0 0 1"/>
-  <parent link="base_link"/>
-  <child link="front_wheel_left"/>
-  <origin rpy="-1.5708 0 0" xyz="0.29 0.265 -0.48"/>
- </joint>
- <link name="front_wheel_right">
-   <visual>
+</link>
+  <link name="laser">
+   <collision>
+    <origin xyz="0 0 0" rpy="0 0 0"/>
     <geometry>
-     <cylinder length="0.06" radius="0.16"/>
-    </geometry>
-    <material name="black"/>
-   </visual>
-   <collision>
-    <geometry>
-     <cylinder length="0.06" radius="0.16"/>
+     <box size="0.1 0.1 0.1"/>
     </geometry>
    </collision>
    <inertial>
-    <mass value="1.0" />
-    <inertia ixx="0.1" iyy="0.1" izz="0.1" ixy="0" ixz="0" iyz="0" />
+    <mass value="1e-5" />
+    <origin xyz="0 0 0" rpy="0 0 0"/>
+    <inertia ixx="1e-6" ixy="0" ixz="0" iyy="1e-6" iyz="0" izz="1e-6" />
    </inertial>
   </link>
- <joint name="front_wheel_right_joint" type="continuous">
-  <axis xyz="0 0 1"/>
-  <parent link="base_link"/>
-  <child link="front_wheel_right"/>
-  <origin rpy="-1.5708 0 0" xyz="0.29 -0.265 -0.48"/>
- </joint>
- <gazebo>
-  <plugin name="differential_drive_controller" filename="libgazebo_ros_diff_drive.so">
-   <legacyMode>false</legacyMode>
-   <leftJoint>front_wheel_left_joint</leftJoint>
-   <rightJoint>front_wheel_right_joint</rightJoint>
-   <robotBaseFrame>base_link</robotBaseFrame>
-   <wheelSeperation>0.50</wheelSeperation>
-   <wheelDiameter>0.32</wheelDiameter>
-   <publishWheelJointState>true</publishWheelJointState>
-  </plugin>
- </gazebo>
- <gazebo>
-  <plugin name="joint_state_publisher" filename="libgazebo_ros_joint_state_publisher.so">
-   <jointName>front_wheel_left_joint, front_wheel_right_joint</jointName>
-  </plugin>
- </gazebo>
- <!--Hokuyo Laser-->
-  <link name="hokuyo">
-    <collision>
-      <origin xyz="0 0 0" rpy="0 0 0"/>
-      <geometry>
-       <box size="0.1 0.1 0.1"/>
-      </geometry>
-    </collision>
-    <visual>
-      <origin xyz="0 0 0" rpy="0 0 0"/>
-      <geometry>
-        <mesh filename="package://mybot_description/meshes/hokuyo.dae"/>
-      </geometry>
-    </visual>
-    <inertial>
-      <mass value="1e-5" />
-      <origin xyz="0 0 0" rpy="0 0 0"/>
-      <inertia ixx="1e-6" ixy="0" ixz="0" iyy="1e-6" iyz="0" izz="1e-6" />
-    </inertial>
-  </link>
-  <gazebo reference="hokuyo">
-   <sensor type="ray" name="hokuyo">
-    <pose>0 0 0 0 0 0</pose>
-    <visualize>true</visualize>
-    <update_rate>40</update_rate>
-    <ray>
-     <scan>
-      <horizontal>
-       <samples>720</samples>
-       <resolution>1</resolution>
-       <min_angle>-2</min_angle>
-       <max_angle>2</max_angle>
-      </horizontal>
-     </scan>
-     <range>
-      <min>0.10</min>
-      <max>6.0</max>
-      <resolution>0.01</resolution>
-     </range>
-    </ray>
-    <plugin name="laser" filename="libgazebo_ros_laser.so">
-     <topicName>/scan</topicName>
-     <frameName>hokuyo</frameName>
-    </plugin>
-   </sensor>
-  </gazebo>
-  <joint name="hokuyo_joint" type="fixed">
+  <joint name="laser_joint" type="fixed">
     <axis xyz="0 1 0" />
     <origin xyz="0.31 0 0" rpy="0 0 0"/>
     <parent link="base_link"/>
-    <child link="hokuyo"/>
+    <child link="laser"/>
   </joint>
 </robot>

Commit message: laser filters and lidar integration

File: mybot_description/urdf/rolstoelbot.xacro (robot description, xacro)
@@ -21,5 +21,5 @@
   </inertial>
 </link>
-  <link name="laser">
+  <!--link name="laser">
    <collision>
     <origin xyz="0 0 0" rpy="0 0 0"/>
@@ -39,4 +39,4 @@
     <parent link="base_link"/>
     <child link="laser"/>
-  </joint>
+  </joint-->
 </robot>

Commit message: Code Comments

File: mybot_description/urdf/rolstoelbot.xacro (robot description, xacro)
@@ -21,22 +21,3 @@
   </inertial>
 </link>
-  <!--link name="laser">
-   <collision>
-    <origin xyz="0 0 0" rpy="0 0 0"/>
-    <geometry>
-     <box size="0.1 0.1 0.1"/>
-    </geometry>
-   </collision>
-   <inertial>
-    <mass value="1e-5" />
-    <origin xyz="0 0 0" rpy="0 0 0"/>
-    <inertia ixx="1e-6" ixy="0" ixz="0" iyy="1e-6" iyz="0" izz="1e-6" />
-   </inertial>
-  </link>
-  <joint name="laser_joint" type="fixed">
-    <axis xyz="0 1 0" />
-    <origin xyz="0.31 0 0" rpy="0 0 0"/>
-    <parent link="base_link"/>
-    <child link="laser"/>
-  </joint-->
 </robot>
